Commit message: feat: integrate controller SIL and harden OpenRB startup
Add shared controller parity and HIL infrastructure, ROS 2 simulation interfaces, companion transport and session tooling, and deployment documentation. Fix the OpenRB control-task stack overflow, retain fatal Cortex context, bound I2C transactions, and expose diagnostics through the shared protocol and CLI.

File: robot_ros_simulation/HexNav_description/urdf/assemblies/HexNav.urdf.xacro (robot description, xacro)
@@ -2,4 +2,13 @@
 <robot xmlns:xacro="http://www.ros.org/wiki/xacro" name="HexNav_macro">
   <xacro:macro name="HexNav" params="prefix">
+  <!-- Massless kinematic root: KDL rejects inertia on the tree root, and the
+       SIL odometry TF (odom -> base_footprint) needs a dedicated root frame
+       that robot_state_publisher does not also parent. -->
+  <link name="${prefix}base_footprint"/>
+  <joint name="${prefix}base_footprint_joint" type="fixed">
+    <parent link="${prefix}base_footprint"/>
+    <child link="${prefix}base_link"/>
+    <origin xyz="0 0 0" rpy="0 0 0"/>
+  </joint>
   <link name="${prefix}base_link">
       <inertial>
